Commit message: Finished "Simulate your robot with gazebo" in Udemy_1

File: Udemy_1/ros3_ws/src/my_robot_description/urdf/common_properties.xacro (robot description, xacro)
@@ -10,3 +10,30 @@
             <color rgba="1 0 0 1" />
         </material>
+        <xacro:macro name="box_inertia" params="m x y z o_xyz o_rpy">
+            <inertial>
+                <mass value="${m}" />
+                <origin xyz="${o_xyz}" rpy="${o_rpy}" />
+                <inertia ixx="${(m/12) *(y*y + z*z)}" ixy="0" ixz="0"
+                         iyy="${(m/12) *(x*x + z*z)}" iyz="0"
+                         izz="${(m/12) *(x*x + y*y)}" />
+            </inertial>
+        </xacro:macro>
+         <xacro:macro name="cylinder_inertia" params="m r l o_xyz o_rpy">
+            <inertial>
+                <mass value="${m}" />
+                <origin xyz="${o_xyz}" rpy="${o_rpy}" />
+                <inertia ixx="${(m/12) *(3 * r * r + l * l)}" ixy="0" ixz="0"
+                         iyy="${(m/12) *(3 * r * r + l*l)}" iyz="0"
+                         izz="${(m/2) * r * r}" />
+            </inertial>
+        </xacro:macro>
+         <xacro:macro name="sphere_inertia" params="m r o_xyz o_rpy">
+            <inertial>
+                <mass value="${m}" />
+                <origin xyz="${o_xyz}" rpy="${o_rpy}" />
+                <inertia ixx="${(m/5) *(2 * r * r)}" ixy="0" ixz="0"
+                         iyy="${(m/5) *(2 * r * r)}" iyz="0"
+                         izz="${(m/5) *(2 * r * r)}" />
+            </inertial>
+        </xacro:macro>
 </robot>

File: Udemy_1/ros3_ws/src/my_robot_description/urdf/mobile_base.xacro (robot description, xacro)
@@ -15,4 +15,12 @@
                 <material name="grey" />
             </visual>
+            <collision>
+                <geometry>
+                    <sphere radius="${wheel_radius}" />
+                </geometry>
+                <origin xyz="0 0 0" rpy="0 0 0" />
+            </collision>
+            <xacro:cylinder_inertia m="1.0" r="${wheel_radius}" l="${wheel_length}"
+                                    o_xyz="0 0 0" o_rpy="0 0 0" />
         </link>
     </xacro:macro>
@@ -26,4 +34,12 @@
             <material name="green" />
         </visual>
+        <collision>
+            <geometry>
+                <box size="${base_length} ${base_width} ${base_height}"/>
+            </geometry>
+            <origin xyz="0 0 0" rpy="0 0 0" />
+        </collision>
+        <xacro:box_inertia m="5.0" x="${base_length}" y="${base_width}" z="${base_height}"
+                           o_xyz="0 0 0" o_rpy="0 0 0" />
     </link>
     <xacro:wheel_link prefix="right" />
@@ -32,9 +48,17 @@
         <visual>
             <geometry>
-                <sphere radius="0.05" />
+                <sphere radius="${wheel_radius / 2.0}" />
             </geometry>
             <origin xyz="0 0 0" rpy="0 0 0" />
             <material name="red" />
         </visual>
+        <collision>
+            <geometry>
+                <sphere radius="${wheel_radius / 2.0}" />
+            </geometry>
+            <origin xyz="0 0 0" rpy="0 0 0" />
+        </collision>
+        <xacro:sphere_inertia m="0.5" r="${wheel_radius / 2.0}"
+                              o_xyz="0 0 0" o_rpy="0 0 0" />
     </link>
     <joint name="base_joint" type="fixed">

File: Udemy_1/ros3_ws/src/my_robot_description/urdf/my_robot_17.urdf.xacro (robot description, xacro)
@@ -3,3 +3,4 @@
     <xacro:include filename="common_properties.xacro" />
     <xacro:include filename="mobile_base.xacro" />
+    <xacro:include filename="mobile_base_gazebo.xacro" />
 </robot>

Commit message: Finished Udemy_1 course'

File: Udemy_1/ros3_ws/src/my_robot_description/urdf/common_properties.xacro (robot description, xacro)
@@ -9,4 +9,10 @@
         <material name="red">
             <color rgba="1 0 0 1" />
+        </material>
+        <material name="blue">
+            <color rgba="0 0 1 1" />
+        </material>
+        <material name="yellow">
+            <color rgba="1 1 0 1" />
         </material>
         <xacro:macro name="box_inertia" params="m x y z o_xyz o_rpy">

File: Udemy_1/ros3_ws/src/my_robot_description/urdf/my_robot_17.urdf.xacro (robot description, xacro)
@@ -4,4 +4,11 @@
     <xacro:include filename="mobile_base.xacro" />
     <xacro:include filename="mobile_base_gazebo.xacro" />
+    <xacro:include filename="arm.xacro" />
+    <xacro:include filename="arm_gazebo.xacro" />
     <xacro:include filename="camera.xacro" />
+    <joint name="mobile_base_arm_joint" type="fixed">
+        <parent link="base_link" />
+        <child link="arm_base_link" />
+        <origin xyz="0 0 ${base_height/2.0}" rpy="0 0 0" />
+    </joint>
 </robot>
